Commit message: update

File: src/kine/urdf/robot.urdf (robot description, URDF)
Before this commit: robot crane3r, 5 links, 4 joints
Links:
- link base_link: geometry visual mesh filename=package://kine/meshes/Crane3R/4200.obj
- link boom_link: geometry visual mesh filename=package://kine/meshes/Crane3R/7000.obj
- link jib_link: geometry visual mesh filename=package://kine/meshes/Crane3R/5200.obj
