Commit message: update

File: src/kine/urdf/crane3r.urdf (robot description, URDF)
Before this commit: robot crane3r, 5 links, 4 joints
Links:
- removed link world
- added link base
- link base_link: geometry collision cylinder length=4.2 radius=0.5; visual mesh filename=package://kine/meshes/Crane3R/4200.obj
- link boom_link: geometry collision box size=7.0 1 1; visual mesh filename=package://kine/meshes/Crane3R/7000.obj
- link jib_link: geometry collision box size=5.2 1 1; visual mesh filename=package://kine/meshes/Crane3R/5200.obj
Joints:
- added joint base_link-base: type fixed, parent base_link, child base, origin xyz=0 0 0 rpy=0 0 0

Commit message: update

File: src/kine/urdf/crane3r.urdf (robot description, URDF)
Before this commit: robot crane3r, 5 links, 5 joints
Joints:
- removed joint base_link-base
- joint base_joint: parent world -> base

Commit message: update

File: src/kine/urdf/crane3r.urdf (robot description, URDF)
Before this commit: robot crane3r, 5 links, 4 joints
Links:
- removed link base
- added link pedestal_link
- added link world
Joints:
- added joint virtual_joint: type fixed, parent world, child pedestal_link, origin xyz=0 0 0 rpy=0 0 0
- joint base_joint: parent base -> pedestal_link
