Commit message: refactor

File: src/kine_robot_description/urdf/crane3r.urdf (robot description, URDF)
Before this commit: robot crane3r, 6 links, 5 joints
Links:
- removed link pedestal_link
Joints:
- removed joint virtual_joint
- joint base_joint: parent pedestal_link -> world

Commit message: fix urdf mesh paths

File: src/kine_robot_description/urdf/crane3r.urdf (robot description, URDF)
Before this commit: robot crane3r, 5 links, 4 joints
Links:
- link base_link: geometry collision cylinder length=4.2 radius=0.5; visual mesh filename=package://kine_robot_description/meshes/Crane3R/4200.obj
- link boom_link: geometry collision box size=7.0 1 1; visual mesh filename=package://kine_robot_description/meshes/Crane3R/7000.obj
- link jib_link: geometry collision box size=5.2 1 1; visual mesh filename=package://kine_robot_description/meshes/Crane3R/5200.obj

File: src/kine_robot_description/urdf/irb2400.urdf (robot description, URDF)
Before this commit: robot abb_irb2400, 9 links, 8 joints
Links:
- link base_link: geometry collision mesh filename=package://kine_robot_description/meshes/irb2400/collision/b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; visual mesh filename=package://kine_robot_description/meshes/irb2400/visual/base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
- link link_1: geometry collision mesh filename=package://kine_robot_description/meshes/irb2400/collision/l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; visual mesh filename=package://kine_robot_description/meshes/irb2400/visual/link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
- link link_2: geometry collision mesh filename=package://kine_robot_description/meshes/irb2400/collision/l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; visual mesh filename=package://kine_robot_description/meshes/irb2400/visual/link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
- link link_3: geometry collision mesh filename=package://kine_robot_description/meshes/irb2400/collision/l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; visual mesh filename=package://kine_robot_description/meshes/irb2400/visual/link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
- link link_4: geometry collision mesh filename=package://kine_robot_description/meshes/irb2400/collision/l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; visual mesh filename=package://kine_robot_description/meshes/irb2400/visual/link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
- link link_5: geometry collision mesh filename=package://kine_robot_description/meshes/irb2400/collision/l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; visual mesh filename=package://kine_robot_description/meshes/irb2400/visual/link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
- link link_6: geometry collision mesh filename=package://kine_robot_description/meshes/irb2400/collision/l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; visual mesh filename=package://kine_robot_description/meshes/irb2400/visual/link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
